Commit message: finsih the empty room

File: objects_description/bottle/mobility.urdf (robot description, URDF)
Before this commit: robot partnet_83620edd3ecbce0de3bf00cc25b4223, 4 links, 3 joints
Links:
- link link_0: geometry collision mesh filename=package://objects_description/bottle/textured_objs/original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; visual mesh filename=package://objects_description/bottle/textured_objs/original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
- link link_1: geometry collision mesh filename=package://objects_description/bottle/textured_objs/new-1.obj; collision mesh filename=package://objects_description/bottle/textured_objs/new-4.obj
